Commit message: Spring 2 -> Spring 3

File: mon_robot_description/urdf/mon_robot.urdf.xacro (robot description, xacro)
@@ -1,5 +1,5 @@
 <?xml version="1.0"?>
 <robot xmlns:xacro="http://www.ros.org/wiki/xacro" name="atawi_3a3">
-  <!-- LIEN FANTOME obligatoire — base_link ne doit pas avoir d'inertie -->
+  <!-- Lien fantôme obligatoire -->
   <link name="world"/>
   <joint name="world_to_base" type="fixed">
@@ -8,42 +8,256 @@
     <origin xyz="0 0 0" rpy="0 0 0"/>
   </joint>
-  <!-- ici commence ton base_link existant -->
+  <!-- ========== BASE / CORPS PRINCIPAL ========== -->
   <link name="base_link">
     <visual>
       <origin xyz="0 0 0" rpy="0 0 0"/>
       <geometry>
-        <box size ="0.3 0.3 0.1"/>
-      </geometry>
-      <material name="chassis_gray">
-        <color rgba="0.5 0.5 0.5 1"/>
+        <mesh filename="package://mon_robot_description/meshes/Body.stl"
+              scale="1 1 1"/>
+      </geometry>
+      <material name="grey">
+        <color rgba="0.6 0.6 0.6 1"/>
       </material>
     </visual>
     <collision>
-      <origin xyz="0 0 0.05" rpy="0 0 0"/>
-      <geometry>
-        <box size="0.037 0.037 0.099"/>
+      <origin xyz="0 0 0.097" rpy="0 0 0"/>
+      <geometry>
+        <box size="0.112 0.063 0.194"/>
       </geometry>
     </collision>
-  </link>
-  <joint name="lid_joint" type="fixed">
-    <parent link="base_link"/>
-    <child link="lid_link"/>
-    <origin xyz="0 0 0.08" rpy="0 0 0"/>
-  </joint>
-  <link name="lid_link">
-    <inertial>
-      <origin xyz="0 0 0" rpy="0 0 0"/>
+    <inertial>
+      <origin xyz="0 0 0.097" rpy="0 0 0"/>
       <mass value="0.5"/>
-      <inertia ixx="0.001" ixy="0" ixz="0"
-               iyy="0.001" iyz="0" izz="0.0005"/>
-    </inertial>
-    <visual>
-      <origin xyz="0 0 0" rpy="0 0 0"/>
-      <geometry>
-        <mesh filename="package://mon_robot_description/meshes/Lid.stl"
-              scale="0.001 0.001 0.001"/>
-      </geometry>
-      <material name="lid_dark">
+      <inertia ixx="0.005" ixy="0" ixz="0"
+               iyy="0.005" iyz="0" izz="0.002"/>
+    </inertial>
+  </link>
+  <!-- ========== HANDLE GAUCHE (fixe) ========== -->
+  <joint name="handle1_joint" type="fixed">
+    <parent link="base_link"/>
+    <child link="handle1_link"/>
+    <origin xyz="0 0 0" rpy="0 0 0"/>
+  </joint>
+  <link name="handle1_link">
+    <visual>
+      <geometry>
+        <mesh filename="package://mon_robot_description/meshes/Handle_1.stl"
+              scale="1 1 1"/>
+      </geometry>
+      <material name="dark_grey">
         <color rgba="0.3 0.3 0.3 1"/>
+      </material>
+    </visual>
+    <collision>
+      <geometry><box size="0.010 0.008 0.025"/></geometry>
+    </collision>
+    <inertial>
+      <mass value="0.02"/>
+      <inertia ixx="0.00001" ixy="0" ixz="0"
+               iyy="0.00001" iyz="0" izz="0.00001"/>
+    </inertial>
+  </link>
+  <!-- ========== HANDLE DROIT (fixe) ========== -->
+  <joint name="handle2_joint" type="fixed">
+    <parent link="base_link"/>
+    <child link="handle2_link"/>
+    <origin xyz="0 0 0" rpy="0 0 0"/>
+  </joint>
+  <link name="handle2_link">
+    <visual>
+      <geometry>
+        <mesh filename="package://mon_robot_description/meshes/Handle_2.stl"
+              scale="1 1 1"/>
+      </geometry>
+      <material name="dark_grey2">
+        <color rgba="0.3 0.3 0.3 1"/>
+      </material>
+    </visual>
+    <collision>
+      <geometry><box size="0.010 0.008 0.025"/></geometry>
+    </collision>
+    <inertial>
+      <mass value="0.02"/>
+      <inertia ixx="0.00001" ixy="0" ixz="0"
+               iyy="0.00001" iyz="0" izz="0.00001"/>
+    </inertial>
+  </link>
+  <!-- ========== ECROUS (fixes) ========== -->
+  <joint name="hexnut1_joint" type="fixed">
+    <parent link="base_link"/>
+    <child link="hexnut1_link"/>
+    <origin xyz="0 0 0" rpy="0 0 0"/>
+  </joint>
+  <link name="hexnut1_link">
+    <visual>
+      <geometry>
+        <mesh filename="package://mon_robot_description/meshes/Hexnut_1.stl"
+              scale="1 1 1"/>
+      </geometry>
+      <material name="metal">
+        <color rgba="0.8 0.7 0.2 1"/>
+      </material>
+    </visual>
+    <inertial>
+      <mass value="0.005"/>
+      <inertia ixx="0.000001" ixy="0" ixz="0"
+               iyy="0.000001" iyz="0" izz="0.000001"/>
+    </inertial>
+  </link>
+  <joint name="hexnut2_joint" type="fixed">
+    <parent link="base_link"/>
+    <child link="hexnut2_link"/>
+    <origin xyz="0 0 0" rpy="0 0 0"/>
+  </joint>
+  <link name="hexnut2_link">
+    <visual>
+      <geometry>
+        <mesh filename="package://mon_robot_description/meshes/Hexnut_2.stl"
+              scale="1 1 1"/>
+      </geometry>
+      <material name="metal2">
+        <color rgba="0.8 0.7 0.2 1"/>
+      </material>
+    </visual>
+    <inertial>
+      <mass value="0.005"/>
+      <inertia ixx="0.000001" ixy="0" ixz="0"
+               iyy="0.000001" iyz="0" izz="0.000001"/>
+    </inertial>
+  </link>
+  <!-- ========== VIS (fixes) ========== -->
+  <joint name="vis1_joint" type="fixed">
+    <parent link="base_link"/>
+    <child link="vis1_link"/>
+    <origin xyz="0 0 0" rpy="0 0 0"/>
+  </joint>
+  <link name="vis1_link">
+    <visual>
+      <geometry>
+        <mesh filename="package://mon_robot_description/meshes/Vis_1.stl"
+              scale="1 1 1"/>
+      </geometry>
+      <material name="silver">
+        <color rgba="0.75 0.75 0.75 1"/>
+      </material>
+    </visual>
+    <inertial>
+      <mass value="0.003"/>
+      <inertia ixx="0.000001" ixy="0" ixz="0"
+               iyy="0.000001" iyz="0" izz="0.000001"/>
+    </inertial>
+  </link>
+  <joint name="vis2_joint" type="fixed">
+    <parent link="base_link"/>
+    <child link="vis2_link"/>
+    <origin xyz="0 0 0" rpy="0 0 0"/>
+  </joint>
+  <link name="vis2_link">
+    <visual>
+      <geometry>
+        <mesh filename="package://mon_robot_description/meshes/Vis_2.stl"
+              scale="1 1 1"/>
+      </geometry>
+      <material name="silver2">
+        <color rgba="0.75 0.75 0.75 1"/>
+      </material>
+    </visual>
+    <inertial>
+      <mass value="0.003"/>
+      <inertia ixx="0.000001" ixy="0" ixz="0"
+               iyy="0.000001" iyz="0" izz="0.000001"/>
+    </inertial>
+  </link>
+  <!-- ========== L2 PIECES (fixes) ========== -->
+  <joint name="l2_1_joint" type="fixed">
+    <parent link="base_link"/>
+    <child link="l2_1_link"/>
+    <origin xyz="0 0 0" rpy="0 0 0"/>
+  </joint>
+  <link name="l2_1_link">
+    <visual>
+      <geometry>
+        <mesh filename="package://mon_robot_description/meshes/L2_1.stl" scale="1 1 1"/>
+      </geometry>
+      <material name="blue"><color rgba="0.2 0.4 0.8 1"/></material>
+    </visual>
+    <inertial>
+      <mass value="0.001"/>
+      <inertia ixx="0.0000001" ixy="0" ixz="0"
+               iyy="0.0000001" iyz="0" izz="0.0000001"/>
+    </inertial>
+  </link>
+  <joint name="l2_2_joint" type="fixed">
+    <parent link="base_link"/>
+    <child link="l2_2_link"/>
+    <origin xyz="0 0 0" rpy="0 0 0"/>
+  </joint>
+  <link name="l2_2_link">
+    <visual>
+      <geometry>
+        <mesh filename="package://mon_robot_description/meshes/L2_2.stl" scale="1 1 1"/>
+      </geometry>
+      <material name="blue2"><color rgba="0.2 0.4 0.8 1"/></material>
+    </visual>
+    <inertial>
+      <mass value="0.001"/>
+      <inertia ixx="0.0000001" ixy="0" ixz="0"
+               iyy="0.0000001" iyz="0" izz="0.0000001"/>
+    </inertial>
+  </link>
+  <joint name="l2_3_joint" type="fixed">
+    <parent link="base_link"/>
+    <child link="l2_3_link"/>
+    <origin xyz="0 0 0" rpy="0 0 0"/>
+  </joint>
+  <link name="l2_3_link">
+    <visual>
+      <geometry>
+        <mesh filename="package://mon_robot_description/meshes/L2_3.stl" scale="1 1 1"/>
+      </geometry>
+      <material name="blue3"><color rgba="0.2 0.4 0.8 1"/></material>
+    </visual>
+    <inertial>
+      <mass value="0.001"/>
+      <inertia ixx="0.0000001" ixy="0" ixz="0"
+               iyy="0.0000001" iyz="0" izz="0.0000001"/>
+    </inertial>
+  </link>
+  <joint name="l2_4_joint" type="fixed">
+    <parent link="base_link"/>
+    <child link="l2_4_link"/>
+    <origin xyz="0 0 0" rpy="0 0 0"/>
+  </joint>
+  <link name="l2_4_link">
+    <visual>
+      <geometry>
+        <mesh filename="package://mon_robot_description/meshes/L2_4.stl" scale="1 1 1"/>
+      </geometry>
+      <material name="blue4"><color rgba="0.2 0.4 0.8 1"/></material>
+    </visual>
+    <inertial>
+      <mass value="0.001"/>
+      <inertia ixx="0.0000001" ixy="0" ixz="0"
+               iyy="0.0000001" iyz="0" izz="0.0000001"/>
+    </inertial>
+  </link>
+  <!-- ========== JOINT 1 — TETE (part2) ROTATION PRINCIPALE ========== -->
+  <joint name="joint1_head" type="revolute">
+    <parent link="base_link"/>
+    <child link="head_link"/>
+    <origin xyz="0 0 0" rpy="0 0 0"/>
+    <axis xyz="0 0 1"/>
+    <limit lower="-3.14159" upper="3.14159"
+           effort="10.0" velocity="1.0"/>
+    <dynamics damping="0.3" friction="0.05"/>
+  </joint>
+  <link name="head_link">
+    <visual>
+      <geometry>
+        <mesh filename="package://mon_robot_description/meshes/part2.stl"
+              scale="1 1 1"/>
+      </geometry>
+      <material name="blue_head">
+        <color rgba="0.2 0.4 0.9 1"/>
       </material>
     </visual>
@@ -51,193 +265,120 @@
       <origin xyz="0 0 0" rpy="0 0 0"/>
       <geometry>
-        <box size="0.037 0.037 0.01"/>
+        <box size="0.101 0.043 0.039"/>
       </geometry>
     </collision>
-  </link>
-  <joint name="grid_joint" type="fixed">
-    <parent link="base_link"/>
-    <child link="grid_link"/>
-    <origin xyz="0 0 0.06" rpy="0 0 0"/>
-  </joint>
-  <link name="grid_link">
-    <inertial>
-      <origin xyz="0 0 0" rpy="0 0 0"/>
-      <mass value="0.2"/>
-      <inertia ixx="0.0005" ixy="0" ixz="0"
-               iyy="0.0005" iyz="0" izz="0.0002"/>
-    </inertial>
-    <visual>
-      <origin xyz="0 0 0" rpy="0 0 0"/>
-      <geometry>
-        <mesh filename="package://mon_robot_description/meshes/Grid.stl"
-              scale="0.001 0.001 0.001"/>
-      </geometry>
-      <material name="grid_blue">
-        <color rgba="0.2 0.2 0.8 0.7"/>
-      </material>
-    </visual>
-    <collision>
-      <origin xyz="0 0 0" rpy="0 0 0"/>
-      <geometry>
-        <box size="0.037 0.037 0.005"/>
-      </geometry>
-    </collision>
-  </link>
-  <joint name="frontal_joint" type="fixed">
-    <parent link="base_link"/>
-    <child link="frontal_link"/>
-    <origin xyz="0.02 0 0.05" rpy="0 0 0"/>
-  </joint>
-  <link name="frontal_link">
-    <inertial>
-      <origin xyz="0 0 0" rpy="0 0 0"/>
-      <mass value="1.0"/>
-      <inertia ixx="0.005" ixy="0" ixz="0"
-               iyy="0.005" iyz="0" izz="0.003"/>
-    </inertial>
-    <visual>
-      <origin xyz="0 0 0" rpy="0 0 0"/>
-      <geometry>
-        <mesh filename="package://mon_robot_description/meshes/frontal_part2.stl"
-              scale="0.001 0.001 0.001"/>
-      </geometry>
-      <material name="frontal_red">
-        <color rgba="1 0 0 0.9"/>
-      </material>
-    </visual>
-    <collision>
-      <origin xyz="0 0 0" rpy="0 0 0"/>
-      <geometry>
-        <box size="0.02 0.037 0.05"/>
-      </geometry>
-    </collision>
-  </link>
-  <joint name="joint1_rotation" type="revolute">
-    <parent link="base_link"/>
-    <child link="link1"/>
-    <origin xyz="0 0 0.10" rpy="0 0 0"/>
+    <inertial>
+      <mass value="0.15"/>
+      <inertia ixx="0.0002" ixy="0" ixz="0"
+               iyy="0.0002" iyz="0" izz="0.0001"/>
+    </inertial>
+  </link>
+  <!-- ========== JOINT 2 — ROTOR (impeller) ROTATION ========== -->
+  <joint name="joint2_rotor" type="revolute">
+    <parent link="head_link"/>
+    <child link="rotor_link"/>
+    <origin xyz="0 0 0" rpy="0 0 0"/>
     <axis xyz="0 0 1"/>
     <limit lower="-3.14159" upper="3.14159"
-           effort="50" velocity="1.0"/>
-    <dynamics damping="0.5" friction="0.1"/>
-  </joint>
-  <link name="link1">
-    <inertial>
-      <origin xyz="0 0 0.1" rpy="0 0 0"/>
-      <mass value="1.5"/>
-      <inertia ixx="0.01" ixy="0" ixz="0"
-               iyy="0.01" iyz="0" izz="0.005"/>
-    </inertial>
-    <visual>
-      <origin xyz="0 0 0.1" rpy="0 0 0"/>
-      <geometry>
-        <cylinder radius="0.03" length="0.2"/>
-      </geometry>
-      <material name="link_orange">
-        <color rgba="1 0.65 0 1"/>
+           effort="5.0" velocity="10.0"/>
+    <dynamics damping="0.1" friction="0.01"/>
+  </joint>
+  <link name="rotor_link">
+    <visual>
+      <geometry>
+        <mesh filename="package://mon_robot_description/meshes/Blade_1.stl"
+              scale="1 1 1"/>
+      </geometry>
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
Commit message: Fix Gazebo simulation launch: model:// mesh URIs for Gazebo and safe GZ_SIM_RESOURCE_PATH
Co-Authored-By: Karl Foko <karlfoko01@gmail.com>

File: mon_robot_description/urdf/mon_robot.urdf.xacro (robot description, xacro)
@@ -1,4 +1,12 @@
 <?xml version="1.0"?>
 <robot xmlns:xacro="http://www.ros.org/wiki/xacro" name="atawi_3a3">
+  <!-- Mesh URI prefix: package:// for RViz, model:// for Gazebo (resolved via GZ_SIM_RESOURCE_PATH) -->
+  <xacro:arg name="use_gazebo" default="false"/>
+  <xacro:if value="$(arg use_gazebo)">
+    <xacro:property name="mesh_uri" value="model://mon_robot_description/meshes"/>
+  </xacro:if>
+  <xacro:unless value="$(arg use_gazebo)">
+    <xacro:property name="mesh_uri" value="package://mon_robot_description/meshes"/>
+  </xacro:unless>
   <!-- Lien fantôme obligatoire -->
   <link name="world"/>
@@ -13,5 +21,5 @@
       <origin xyz="0 0 0" rpy="0 0 0"/>
       <geometry>
-        <mesh filename="package://mon_robot_description/meshes/Body.stl"
+        <mesh filename="${mesh_uri}/Body.stl"
               scale="1 1 1"/>
       </geometry>
@@ -42,5 +50,5 @@
     <visual>
       <geometry>
-        <mesh filename="package://mon_robot_description/meshes/Handle_1.stl"
+        <mesh filename="${mesh_uri}/Handle_1.stl"
               scale="1 1 1"/>
       </geometry>
@@ -67,5 +75,5 @@
     <visual>
       <geometry>
-        <mesh filename="package://mon_robot_description/meshes/Handle_2.stl"
+        <mesh filename="${mesh_uri}/Handle_2.stl"
               scale="1 1 1"/>
       </geometry>
@@ -92,5 +100,5 @@
     <visual>
       <geometry>
-        <mesh filename="package://mon_robot_description/meshes/Hexnut_1.stl"
+        <mesh filename="${mesh_uri}/Hexnut_1.stl"
               scale="1 1 1"/>
       </geometry>
@@ -113,5 +121,5 @@
     <visual>
       <geometry>
-        <mesh filename="package://mon_robot_description/meshes/Hexnut_2.stl"
+        <mesh filename="${mesh_uri}/Hexnut_2.stl"
               scale="1 1 1"/>
       </geometry>
@@ -135,5 +143,5 @@
     <visual>
       <geometry>
-        <mesh filename="package://mon_robot_description/meshes/Vis_1.stl"
+        <mesh filename="${mesh_uri}/Vis_1.stl"
               scale="1 1 1"/>
       </geometry>
@@ -156,5 +164,5 @@
     <visual>
       <geometry>
-        <mesh filename="package://mon_robot_description/meshes/Vis_2.stl"
+        <mesh filename="${mesh_uri}/Vis_2.stl"
               scale="1 1 1"/>
       </geometry>
@@ -178,5 +186,5 @@
     <visual>
       <geometry>
-        <mesh filename="package://mon_robot_description/meshes/L2_1.stl" scale="1 1 1"/>
+        <mesh filename="${mesh_uri}/L2_1.stl" scale="1 1 1"/>
       </geometry>
       <material name="blue"><color rgba="0.2 0.4 0.8 1"/></material>
@@ -196,5 +204,5 @@
     <visual>
       <geometry>
-        <mesh filename="package://mon_robot_description/meshes/L2_2.stl" scale="1 1 1"/>
+        <mesh filename="${mesh_uri}/L2_2.stl" scale="1 1 1"/>
       </geometry>
       <material name="blue2"><color rgba="0.2 0.4 0.8 1"/></material>
@@ -214,5 +222,5 @@
     <visual>
       <geometry>
-        <mesh filename="package://mon_robot_description/meshes/L2_3.stl" scale="1 1 1"/>
+        <mesh filename="${mesh_uri}/L2_3.stl" scale="1 1 1"/>
       </geometry>
       <material name="blue3"><color rgba="0.2 0.4 0.8 1"/></material>
@@ -232,5 +240,5 @@
     <visual>
       <geometry>
-        <mesh filename="package://mon_robot_description/meshes/L2_4.stl" scale="1 1 1"/>
+        <mesh filename="${mesh_uri}/L2_4.stl" scale="1 1 1"/>
       </geometry>
       <material name="blue4"><color rgba="0.2 0.4 0.8 1"/></material>
@@ -255,5 +263,5 @@
     <visual>
       <geometry>
-        <mesh filename="package://mon_robot_description/meshes/part2.stl"
+        <mesh filename="${mesh_uri}/part2.stl"
               scale="1 1 1"/>
       </geometry>
@@ -287,5 +295,5 @@
     <visual>
       <geometry>
-        <mesh filename="package://mon_robot_description/meshes/Blade_1.stl"
+        <mesh filename="${mesh_uri}/Blade_1.stl"
               scale="1 1 1"/>
       </geometry>
@@ -312,5 +320,5 @@
     <visual>
       <geometry>
-        <mesh filename="package://mon_robot_description/meshes/Blade_2.stl" scale="1 1 1"/>
+        <mesh filename="${mesh_uri}/Blade_2.stl" scale="1 1 1"/>
       </geometry>
       <material name="blade2"><color rgba="0.9 0.4 0.1 1"/></material>
@@ -330,5 +338,5 @@
     <visual>
       <geometry>
-        <mesh filename="package://mon_robot_description/meshes/Blade_3.stl" scale="1 1 1"/>
+        <mesh filename="${mesh_uri}/Blade_3.stl" scale="1 1 1"/>
       </geometry>
       <material name="blade3"><color rgba="0.9 0.4 0.1 1"/></material>
@@ -348,5 +356,5 @@
     <visual>
       <geometry>
-        <mesh filename="package://mon_robot_description/meshes/Blade_4.stl" scale="1 1 1"/>
+        <mesh filename="${mesh_uri}/Blade_4.stl" scale="1 1 1"/>
       </geometry>
       <material name="blade4"><color rgba="0.9 0.4 0.1 1"/></material>
@@ -375,5 +383,6 @@
     </inertial>
   </link>
-  <!-- ========== ROS2 CONTROL ========== -->
+  <!-- ========== ROS2 CONTROL (Gazebo uniquement) ========== -->
+  <xacro:if value="$(arg use_gazebo)">
   <ros2_control name="GazeboSystem" type="system">
     <hardware>
@@ -405,3 +414,4 @@
     </plugin>
   </gazebo>
+  </xacro:if>
 </robot>
