Commit message: fix: align boat model and restore gazebo simulation

File: mon_robot_description/urdf/mon_robot.urdf.xacro (robot description, xacro)
@@ -4,7 +4,6 @@
   <xacro:arg name="use_gazebo" default="false"/>
   <xacro:arg name="controllers_yaml" default=""/>
-  <!-- Facteur d'echelle global du device. Changez cette seule valeur pour
-       redimensionner tout le robot (meshes + collisions + offsets). -->
-  <xacro:property name="s" value="10.0"/>
+  <!-- Facteur d'echelle global du device. 1.0 conserve la taille native des STL. -->
+  <xacro:property name="s" value="1.0"/>
   <xacro:if value="$(arg use_gazebo)">
     <xacro:property name="mesh_uri" value="model://mon_robot_description/meshes"/>
@@ -16,5 +15,5 @@
        trajectoire n'est commandee (seuls joint1_head/joint2_rotor bougent).
        Le lien "world" sert aussi de repere fixe en RViz.
-       world_to_hull origin z : hauteur de la coque par rapport a l'eau (z=0). -->
+       world_to_hull origin z : hauteur du repere technique par rapport a l'eau (z=0). -->
   <link name="world"/>
   <joint name="world_to_hull" type="fixed">
@@ -23,22 +22,8 @@
     <origin xyz="0 0 0.15" rpy="0 0 0"/>
   </joint>
-  <!-- ========== COQUE (corps porteur, large et plat) ==========
-       Posee a plat sur l'eau, dimensionnee pour porter le device (x10). -->
+  <!-- ========== REPERE TECHNIQUE INVISIBLE ==========
+       hull_link reste present pour conserver les frames ROS/Gazebo, mais il
+       n'a plus de visual/collision afin de supprimer le carre noir dans Gazebo. -->
   <link name="hull_link">
-    <visual>
-      <origin xyz="0 0 0" rpy="0 0 0"/>
-      <geometry>
-        <box size="2.4 1.2 0.4"/>
-      </geometry>
-      <material name="hull">
-        <color rgba="0.15 0.20 0.30 1"/>
-      </material>
-    </visual>
-    <collision>
-      <origin xyz="0 0 0" rpy="0 0 0"/>
-      <geometry>
-        <box size="2.4 1.2 0.4"/>
-      </geometry>
-    </collision>
     <inertial>
       <origin xyz="0 0 -0.10" rpy="0 0 0"/>
@@ -48,13 +33,13 @@
     </inertial>
   </link>
-  <!-- Robot couche a l'horizontale et pose sur le pont de la coque.
-       rpy="0 -pi/2 0" : l'axe long du device (+Z) pointe vers l'avant (+X).
-       Ajustez l'origin xyz pour repositionner le robot sur le pont. -->
+  <!-- Robot STL recentre et couche a l'horizontale sur la surface d'eau.
+       xyz compense l'origine interne des STL. rpy aligne l'axe long du device
+       avec l'horizon et remet l'axe vertical du STL vers le haut. -->
   <joint name="hull_to_base" type="fixed">
     <parent link="hull_link"/>
     <child link="base_link"/>
-    <origin xyz="-0.7 0 0.45" rpy="0 -1.5708 0"/>
-  </joint>
-  <!-- ========== BASE / CORPS PRINCIPAL (device, pose sur la coque) ========== -->
+    <origin xyz="-1.2805 -0.6259 -0.9647" rpy="1.5708 0 1.5708"/>
+  </joint>
+  <!-- ========== BASE / CORPS PRINCIPAL (device) ========== -->
   <link name="base_link">
     <visual>
