Commit message: Flottaison horizontale, course temporelle et robustesse
Simulation Gazebo:
- Base libre en simulation (lien world rendu conditionnel via xacro, RViz uniquement)
- Plugin Buoyancy gradue + surface d'eau sans collision -> flottaison reelle
- Centre de masse abaisse (lestage) -> stabilite horizontale type bouee
- Spawn horizontal (pitch=0) proche de l'equilibre de flottaison (boat_z=-0.1)
- Odometrie 3D du bateau (OdometryPublisher) bridgee et enregistree au rosbag
- Controleurs demarres sur fin de spawn (RegisterEventHandler) vs delai fixe fragile
- Plugins systeme Gazebo Harmonic ajoutes (Physics/SceneBroadcaster/UserCommands)

Corrections:
- Declaration de parametres idempotente (plus de crash 'use_sim_time' deja declare)
- workspace_yaw_samples couvre tout le cercle [-pi, pi] (test corrige)
- display/test_display.launch: ParameterValue(value_type=str) + API non depreciee
- generate_placeholder_meshes non destructif (n'ecrase plus les meshes CAO)

Nettoyage:
- Bloc PID 'gains' mort retire de controllers.yaml (interface position)
- Dependances inutilisees retirees (sensor_msgs/geometry_msgs), nav_msgs ajoutee
- Documentation projet.md mise a jour (flottaison, course temporelle, base libre)

Co-Authored-By: Claude Opus 4.8 <noreply@anthropic.com>

File: mon_robot_description/urdf/mon_robot.urdf.xacro (robot description, xacro)
@@ -10,11 +10,14 @@
     <xacro:property name="mesh_uri" value="package://mon_robot_description/meshes"/>
   </xacro:unless>
-  <!-- Lien fantôme obligatoire -->
-  <link name="world"/>
-  <joint name="world_to_base" type="fixed">
-    <parent link="world"/>
-    <child link="base_link"/>
-    <origin xyz="0 0 0" rpy="0 0 0"/>
-  </joint>
+  <!-- Lien "world" UNIQUEMENT hors Gazebo (RViz a besoin d'un repere fixe).
+       En Gazebo, la base reste LIBRE pour pouvoir flotter (pas de joint fixe). -->
+  <xacro:unless value="$(arg use_gazebo)">
+    <link name="world"/>
+    <joint name="world_to_base" type="fixed">
+      <parent link="world"/>
+      <child link="base_link"/>
+      <origin xyz="0 0 0" rpy="0 0 0"/>
+    </joint>
+  </xacro:unless>
   <!-- ========== BASE / CORPS PRINCIPAL ========== -->
   <link name="base_link">
@@ -36,5 +39,7 @@
     </collision>
     <inertial>
-      <origin xyz="0 0 0.097" rpy="0 0 0"/>
+      <!-- Centre de masse abaisse (lestage / quille) : auto-redressement
+           horizontal une fois a flot, comme une bouee. -->
+      <origin xyz="0 0 0.025" rpy="0 0 0"/>
       <mass value="0.5"/>
       <inertia ixx="0.005" ixy="0" ixz="0"
@@ -414,4 +419,13 @@
       <parameters>$(arg controllers_yaml)</parameters>
     </plugin>
+    <!-- Odometrie 3D du bateau (pose monde -> base_link) pour suivre la
+         flottaison et la course temporelle. Publie /model/atawi_3a3/odometry. -->
+    <plugin filename="gz-sim-odometry-publisher-system"
+            name="gz::sim::systems::OdometryPublisher">
+      <dimensions>3</dimensions>
+      <odom_frame>world</odom_frame>
+      <robot_base_frame>base_link</robot_base_frame>
+      <odom_publish_frequency>50</odom_publish_frequency>
+    </plugin>
   </gazebo>
   </xacro:if>

Commit message: Bateau horizontal sur coque flottante + agrandi x3 + eau retravaillee
- Nouveau corps racine hull_link : coque large et plate (0.70x0.36x0.12,
  ~10 kg, CoM bas) -> flottaison STABLE a l'horizontale (box, supporte par
  le plugin Buoyancy gradue).
- Robot ATAGI-3A3 couche a l'horizontale et pose sur le pont via le joint
  fixe hull_to_base (rpy 0 -pi/2 0) ; base_link n'a plus de collision.
- Modele agrandi x3 (meshes scale 3 3 3, collisions et offsets x3) ~0.57 m.
- world conditionnel -> hull_link (RViz) ; OdometryPublisher suit hull_link.
- Eau : teinte mer turquoise lumineuse + rendu PBR.
- Spawn boat_z=0.05, pitch/roll=0 (coque a plat).
- docs/COMMANDES.md : reference complete des commandes + lien README.
- docs/projet.md mis a jour (coque, x3).

Co-Authored-By: Claude Opus 4.8 <noreply@anthropic.com>

File: mon_robot_description/urdf/mon_robot.urdf.xacro (robot description, xacro)
@@ -11,14 +11,50 @@
   </xacro:unless>
   <!-- Lien "world" UNIQUEMENT hors Gazebo (RViz a besoin d'un repere fixe).
-       En Gazebo, la base reste LIBRE pour pouvoir flotter (pas de joint fixe). -->
+       En Gazebo, la COQUE (hull_link) reste LIBRE pour pouvoir flotter. -->
   <xacro:unless value="$(arg use_gazebo)">
     <link name="world"/>
-    <joint name="world_to_base" type="fixed">
+    <joint name="world_to_hull" type="fixed">
       <parent link="world"/>
-      <child link="base_link"/>
+      <child link="hull_link"/>
       <origin xyz="0 0 0" rpy="0 0 0"/>
     </joint>
   </xacro:unless>
-  <!-- ========== BASE / CORPS PRINCIPAL ========== -->
+  <!-- ========== COQUE FLOTTANTE (corps racine, large et plat) ==========
+       Box large >> haute => flottaison stable a plat. Toute la portance vient
+       d'ici (le plugin Buoyancy gradue ne supporte que box/sphere). Le device
+       est pose dessus, a l'horizontale, au-dessus de l'eau. -->
+  <link name="hull_link">
+    <visual>
+      <origin xyz="0 0 0" rpy="0 0 0"/>
+      <geometry>
+        <box size="0.70 0.36 0.12"/>
+      </geometry>
+      <material name="hull">
+        <color rgba="0.15 0.20 0.30 1"/>
+      </material>
+    </visual>
+    <collision>
+      <origin xyz="0 0 0" rpy="0 0 0"/>
+      <geometry>
+        <box size="0.70 0.36 0.12"/>
+      </geometry>
+    </collision>
+    <inertial>
+      <!-- Masse principale, CoM bas (lestage) => auto-redressement a plat -->
+      <origin xyz="0 0 -0.04" rpy="0 0 0"/>
+      <mass value="10.0"/>
+      <inertia ixx="0.12" ixy="0" ixz="0"
+               iyy="0.42" iyz="0" izz="0.52"/>
+    </inertial>
+  </link>
+  <!-- Robot couche a l'horizontale et pose sur le pont de la coque.
+       rpy="0 -pi/2 0" : l'axe long du device (+Z) pointe vers l'avant (+X),
+       l'helice (joint2_rotor) tourne alors autour de l'axe d'avance. -->
+  <joint name="hull_to_base" type="fixed">
+    <parent link="hull_link"/>
+    <child link="base_link"/>
+    <origin xyz="-0.20 0 0.12" rpy="0 -1.5708 0"/>
+  </joint>
+  <!-- ========== BASE / CORPS PRINCIPAL (device, pose sur la coque) ========== -->
   <link name="base_link">
     <visual>
@@ -26,5 +62,5 @@
       <geometry>
         <mesh filename="${mesh_uri}/Body.stl"
-              scale="1 1 1"/>
+              scale="3 3 3"/>
       </geometry>
       <material name="grey">
@@ -32,14 +68,6 @@
       </material>
     </visual>
-    <collision>
-      <origin xyz="0 0 0.097" rpy="0 0 0"/>
-      <geometry>
-        <box size="0.112 0.063 0.194"/>
-      </geometry>
-    </collision>
-    <inertial>
-      <!-- Centre de masse abaisse (lestage / quille) : auto-redressement
-           horizontal une fois a flot, comme une bouee. -->
-      <origin xyz="0 0 0.025" rpy="0 0 0"/>
+    <inertial>
+      <origin xyz="0 0 0" rpy="0 0 0"/>
       <mass value="0.5"/>
       <inertia ixx="0.005" ixy="0" ixz="0"
@@ -57,5 +85,5 @@
       <geometry>
         <mesh filename="${mesh_uri}/Handle_1.stl"
-              scale="1 1 1"/>
+              scale="3 3 3"/>
       </geometry>
       <material name="dark_grey">
@@ -64,5 +92,5 @@
     </visual>
     <collision>
-      <geometry><box size="0.010 0.008 0.025"/></geometry>
+      <geometry><box size="0.030 0.024 0.075"/></geometry>
     </collision>
     <inertial>
@@ -82,5 +110,5 @@
       <geometry>
         <mesh filename="${mesh_uri}/Handle_2.stl"
-              scale="1 1 1"/>
+              scale="3 3 3"/>
       </geometry>
       <material name="dark_grey2">
@@ -89,5 +117,5 @@
     </visual>
     <collision>
-      <geometry><box size="0.010 0.008 0.025"/></geometry>
+      <geometry><box size="0.030 0.024 0.075"/></geometry>
     </collision>
     <inertial>
@@ -107,5 +135,5 @@
       <geometry>
         <mesh filename="${mesh_uri}/Hexnut_1.stl"
-              scale="1 1 1"/>
+              scale="3 3 3"/>
       </geometry>
       <material name="metal">
@@ -128,5 +156,5 @@
       <geometry>
         <mesh filename="${mesh_uri}/Hexnut_2.stl"
-              scale="1 1 1"/>
+              scale="3 3 3"/>
       </geometry>
       <material name="metal2">
@@ -150,5 +178,5 @@
       <geometry>
         <mesh filename="${mesh_uri}/Vis_1.stl"
-              scale="1 1 1"/>
+              scale="3 3 3"/>
       </geometry>
       <material name="silver">
@@ -171,5 +199,5 @@
       <geometry>
         <mesh filename="${mesh_uri}/Vis_2.stl"
-              scale="1 1 1"/>
+              scale="3 3 3"/>
       </geometry>
       <material name="silver2">
@@ -192,5 +220,5 @@
     <visual>
       <geometry>
-        <mesh filename="${mesh_uri}/L2_1.stl" scale="1 1 1"/>
+        <mesh filename="${mesh_uri}/L2_1.stl" scale="3 3 3"/>
       </geometry>
       <material name="blue"><color rgba="0.2 0.4 0.8 1"/></material>
@@ -210,5 +238,5 @@
     <visual>
       <geometry>
-        <mesh filename="${mesh_uri}/L2_2.stl" scale="1 1 1"/>
+        <mesh filename="${mesh_uri}/L2_2.stl" scale="3 3 3"/>
       </geometry>
       <material name="blue2"><color rgba="0.2 0.4 0.8 1"/></material>
@@ -228,5 +256,5 @@
     <visual>
       <geometry>
-        <mesh filename="${mesh_uri}/L2_3.stl" scale="1 1 1"/>
+        <mesh filename="${mesh_uri}/L2_3.stl" scale="3 3 3"/>
       </geometry>
       <material name="blue3"><color rgba="0.2 0.4 0.8 1"/></material>
@@ -246,5 +274,5 @@
     <visual>
       <geometry>
-        <mesh filename="${mesh_uri}/L2_4.stl" scale="1 1 1"/>
+        <mesh filename="${mesh_uri}/L2_4.stl" scale="3 3 3"/>
       </geometry>
       <material name="blue4"><color rgba="0.2 0.4 0.8 1"/></material>
@@ -270,5 +298,5 @@
       <geometry>
         <mesh filename="${mesh_uri}/part2.stl"
-              scale="1 1 1"/>
+              scale="3 3 3"/>
       </geometry>
       <material name="blue_head">
@@ -279,5 +307,5 @@
       <origin xyz="0 0 0" rpy="0 0 0"/>
       <geometry>
-        <box size="0.101 0.043 0.039"/>
+        <box size="0.303 0.129 0.117"/>
       </geometry>
     </collision>
@@ -302,5 +330,5 @@
       <geometry>
         <mesh filename="${mesh_uri}/Blade_1.stl"
-              scale="1 1 1"/>
+              scale="3 3 3"/>
       </geometry>
       <material name="blade_color">
@@ -309,5 +337,5 @@
     </visual>
     <collision>
-      <geometry><cylinder radius="0.015" length="0.006"/></geometry>
+      <geometry><cylinder radius="0.045" length="0.018"/></geometry>
     </collision>
     <inertial>
@@ -326,5 +354,5 @@
     <visual>
       <geometry>
-        <mesh filename="${mesh_uri}/Blade_2.stl" scale="1 1 1"/>
+        <mesh filename="${mesh_uri}/Blade_2.stl" scale="3 3 3"/>
       </geometry>
       <material name="blade2"><color rgba="0.9 0.4 0.1 1"/></material>
@@ -344,5 +372,5 @@
     <visual>
       <geometry>
-        <mesh filename="${mesh_uri}/Blade_3.stl" scale="1 1 1"/>
+        <mesh filename="${mesh_uri}/Blade_3.stl" scale="3 3 3"/>
       </geometry>
       <material name="blade3"><color rgba="0.9 0.4 0.1 1"/></material>
@@ -362,5 +390,5 @@
     <visual>
       <geometry>
-        <mesh filename="${mesh_uri}/Blade_4.stl" scale="1 1 1"/>
+        <mesh filename="${mesh_uri}/Blade_4.stl" scale="3 3 3"/>
       </geometry>
       <material name="blade4"><color rgba="0.9 0.4 0.1 1"/></material>
@@ -376,9 +404,9 @@
     <parent link="rotor_link"/>
     <child link="tool_link"/>
-    <origin xyz="0 0 0.010" rpy="0 0 0"/>
+    <origin xyz="0 0 0.030" rpy="0 0 0"/>
   </joint>
   <link name="tool_link">
     <visual>
-      <geometry><sphere radius="0.005"/></geometry>
+      <geometry><sphere radius="0.015"/></geometry>
       <material name="red"><color rgba="1 0 0 1"/></material>
     </visual>
@@ -425,5 +453,5 @@
       <dimensions>3</dimensions>
       <odom_frame>world</odom_frame>
-      <robot_base_frame>base_link</robot_base_frame>
+      <robot_base_frame>hull_link</robot_base_frame>
       <odom_publish_frequency>50</odom_publish_frequency>
     </plugin>

Commit message: Bateau fixe a plat sur l'eau, immobile, agrandi x10
- Bateau FIXE au monde (joint world_to_hull toujours present) : pose a plat
  et IMMOBILE tant qu'aucune trajectoire n'est commandee ; seuls joint1_head
  et joint2_rotor bougent.
- Echelle x10 via une propriete xacro unique 's' (meshes + collisions +
  offsets exprimes en fonction de s) -> redimensionnable en un seul endroit.
- Coque agrandie a 2.4 x 1.2 x 0.4 m pour porter le device x10.
- Plugin Buoyancy retire (inutile pour un bateau fixe).
- Hauteur reglee via world_to_hull (z=0.15), boat_z=0 par defaut.
- docs/projet.md mis a jour.

Co-Authored-By: Claude Opus 4.8 <noreply@anthropic.com>

File: mon_robot_description/urdf/mon_robot.urdf.xacro (robot description, xacro)
@@ -4,4 +4,7 @@
   <xacro:arg name="use_gazebo" default="false"/>
   <xacro:arg name="controllers_yaml" default=""/>
+  <!-- Facteur d'echelle global du device. Changez cette seule valeur pour
+       redimensionner tout le robot (meshes + collisions + offsets). -->
+  <xacro:property name="s" value="10.0"/>
   <xacro:if value="$(arg use_gazebo)">
     <xacro:property name="mesh_uri" value="model://mon_robot_description/meshes"/>
@@ -10,23 +13,21 @@
     <xacro:property name="mesh_uri" value="package://mon_robot_description/meshes"/>
   </xacro:unless>
-  <!-- Lien "world" UNIQUEMENT hors Gazebo (RViz a besoin d'un repere fixe).
-       En Gazebo, la COQUE (hull_link) reste LIBRE pour pouvoir flotter. -->
-  <xacro:unless value="$(arg use_gazebo)">
-    <link name="world"/>
-    <joint name="world_to_hull" type="fixed">
-      <parent link="world"/>
-      <child link="hull_link"/>
+  <!-- Bateau FIXE au monde : pose a plat sur l'eau et IMMOBILE tant qu'aucune
+       trajectoire n'est commandee (seuls joint1_head/joint2_rotor bougent).
+       Le lien "world" sert aussi de repere fixe en RViz.
+       world_to_hull origin z : hauteur de la coque par rapport a l'eau (z=0). -->
+  <link name="world"/>
+  <joint name="world_to_hull" type="fixed">
+    <parent link="world"/>
+    <child link="hull_link"/>
+    <origin xyz="0 0 0.15" rpy="0 0 0"/>
+  </joint>
+  <!-- ========== COQUE (corps porteur, large et plat) ==========
+       Posee a plat sur l'eau, dimensionnee pour porter le device (x10). -->
+  <link name="hull_link">
+    <visual>
       <origin xyz="0 0 0" rpy="0 0 0"/>
-    </joint>
-  </xacro:unless>
-  <!-- ========== COQUE FLOTTANTE (corps racine, large et plat) ==========
-       Box large >> haute => flottaison stable a plat. Toute la portance vient
-       d'ici (le plugin Buoyancy gradue ne supporte que box/sphere). Le device
-       est pose dessus, a l'horizontale, au-dessus de l'eau. -->
-  <link name="hull_link">
-    <visual>
-      <origin xyz="0 0 0" rpy="0 0 0"/>
-      <geometry>
-        <box size="0.70 0.36 0.12"/>
+      <geometry>
+        <box size="2.4 1.2 0.4"/>
       </geometry>
       <material name="hull">
@@ -37,22 +38,21 @@
       <origin xyz="0 0 0" rpy="0 0 0"/>
       <geometry>
-        <box size="0.70 0.36 0.12"/>
+        <box size="2.4 1.2 0.4"/>
       </geometry>
     </collision>
     <inertial>
-      <!-- Masse principale, CoM bas (lestage) => auto-redressement a plat -->
-      <origin xyz="0 0 -0.04" rpy="0 0 0"/>
-      <mass value="10.0"/>
-      <inertia ixx="0.12" ixy="0" ixz="0"
-               iyy="0.42" iyz="0" izz="0.52"/>
+      <origin xyz="0 0 -0.10" rpy="0 0 0"/>
+      <mass value="50.0"/>
+      <inertia ixx="6.7" ixy="0" ixz="0"
+               iyy="24.7" iyz="0" izz="30.0"/>
     </inertial>
   </link>
   <!-- Robot couche a l'horizontale et pose sur le pont de la coque.
-       rpy="0 -pi/2 0" : l'axe long du device (+Z) pointe vers l'avant (+X),
-       l'helice (joint2_rotor) tourne alors autour de l'axe d'avance. -->
+       rpy="0 -pi/2 0" : l'axe long du device (+Z) pointe vers l'avant (+X).
+       Ajustez l'origin xyz pour repositionner le robot sur le pont. -->
   <joint name="hull_to_base" type="fixed">
     <parent link="hull_link"/>
     <child link="base_link"/>
-    <origin xyz="-0.20 0 0.12" rpy="0 -1.5708 0"/>
+    <origin xyz="-0.7 0 0.45" rpy="0 -1.5708 0"/>
   </joint>
   <!-- ========== BASE / CORPS PRINCIPAL (device, pose sur la coque) ========== -->
@@ -62,5 +62,5 @@
       <geometry>
         <mesh filename="${mesh_uri}/Body.stl"
-              scale="3 3 3"/>
+              scale="${s} ${s} ${s}"/>
       </geometry>
       <material name="grey">
@@ -85,5 +85,5 @@
       <geometry>
         <mesh filename="${mesh_uri}/Handle_1.stl"
-              scale="3 3 3"/>
+              scale="${s} ${s} ${s}"/>
       </geometry>
       <material name="dark_grey">
@@ -92,5 +92,5 @@
     </visual>
     <collision>
-      <geometry><box size="0.030 0.024 0.075"/></geometry>
+      <geometry><box size="${0.010*s} ${0.008*s} ${0.025*s}"/></geometry>
     </collision>
     <inertial>
@@ -110,5 +110,5 @@
       <geometry>
         <mesh filename="${mesh_uri}/Handle_2.stl"
-              scale="3 3 3"/>
+              scale="${s} ${s} ${s}"/>
       </geometry>
       <material name="dark_grey2">
@@ -117,5 +117,5 @@
     </visual>
     <collision>
-      <geometry><box size="0.030 0.024 0.075"/></geometry>
+      <geometry><box size="${0.010*s} ${0.008*s} ${0.025*s}"/></geometry>
     </collision>
     <inertial>
@@ -135,5 +135,5 @@
       <geometry>
         <mesh filename="${mesh_uri}/Hexnut_1.stl"
-              scale="3 3 3"/>
+              scale="${s} ${s} ${s}"/>
       </geometry>
       <material name="metal">
@@ -156,5 +156,5 @@
       <geometry>
         <mesh filename="${mesh_uri}/Hexnut_2.stl"
-              scale="3 3 3"/>
+              scale="${s} ${s} ${s}"/>
       </geometry>
       <material name="metal2">
@@ -178,5 +178,5 @@
       <geometry>
         <mesh filename="${mesh_uri}/Vis_1.stl"
-              scale="3 3 3"/>
+              scale="${s} ${s} ${s}"/>
       </geometry>
       <material name="silver">
@@ -199,5 +199,5 @@
       <geometry>
         <mesh filename="${mesh_uri}/Vis_2.stl"
-              scale="3 3 3"/>
+              scale="${s} ${s} ${s}"/>
       </geometry>
       <material name="silver2">
@@ -220,5 +220,5 @@
     <visual>
       <geometry>
-        <mesh filename="${mesh_uri}/L2_1.stl" scale="3 3 3"/>
+        <mesh filename="${mesh_uri}/L2_1.stl" scale="${s} ${s} ${s}"/>
       </geometry>
       <material name="blue"><color rgba="0.2 0.4 0.8 1"/></material>
@@ -238,5 +238,5 @@
     <visual>
       <geometry>
-        <mesh filename="${mesh_uri}/L2_2.stl" scale="3 3 3"/>
+        <mesh filename="${mesh_uri}/L2_2.stl" scale="${s} ${s} ${s}"/>
       </geometry>
       <material name="blue2"><color rgba="0.2 0.4 0.8 1"/></material>
@@ -256,5 +256,5 @@
     <visual>
       <geometry>
-        <mesh filename="${mesh_uri}/L2_3.stl" scale="3 3 3"/>
+        <mesh filename="${mesh_uri}/L2_3.stl" scale="${s} ${s} ${s}"/>
       </geometry>
       <material name="blue3"><color rgba="0.2 0.4 0.8 1"/></material>
@@ -274,5 +274,5 @@
     <visual>
       <geometry>
-        <mesh filename="${mesh_uri}/L2_4.stl" scale="3 3 3"/>
+        <mesh filename="${mesh_uri}/L2_4.stl" scale="${s} ${s} ${s}"/>
       </geometry>
       <material name="blue4"><color rgba="0.2 0.4 0.8 1"/></material>
@@ -298,5 +298,5 @@
       <geometry>
         <mesh filename="${mesh_uri}/part2.stl"
-              scale="3 3 3"/>
+              scale="${s} ${s} ${s}"/>
       </geometry>
       <material name="blue_head">
@@ -307,5 +307,5 @@
       <origin xyz="0 0 0" rpy="0 0 0"/>
       <geometry>
-        <box size="0.303 0.129 0.117"/>
+        <box size="${0.101*s} ${0.043*s} ${0.039*s}"/>
       </geometry>
     </collision>
@@ -330,5 +330,5 @@
       <geometry>
         <mesh filename="${mesh_uri}/Blade_1.stl"
-              scale="3 3 3"/>
+              scale="${s} ${s} ${s}"/>
       </geometry>
       <material name="blade_color">
@@ -337,5 +337,5 @@
     </visual>
     <collision>
-      <geometry><cylinder radius="0.045" length="0.018"/></geometry>
+      <geometry><cylinder radius="${0.015*s}" length="${0.006*s}"/></geometry>
     </collision>
     <inertial>
@@ -354,5 +354,5 @@
     <visual>
       <geometry>
-        <mesh filename="${mesh_uri}/Blade_2.stl" scale="3 3 3"/>
+        <mesh filename="${mesh_uri}/Blade_2.stl" scale="${s} ${s} ${s}"/>
       </geometry>
       <material name="blade2"><color rgba="0.9 0.4 0.1 1"/></material>
@@ -372,5 +372,5 @@
     <visual>
       <geometry>
-        <mesh filename="${mesh_uri}/Blade_3.stl" scale="3 3 3"/>
+        <mesh filename="${mesh_uri}/Blade_3.stl" scale="${s} ${s} ${s}"/>
       </geometry>
       <material name="blade3"><color rgba="0.9 0.4 0.1 1"/></material>
@@ -390,5 +390,5 @@
     <visual>
       <geometry>
-        <mesh filename="${mesh_uri}/Blade_4.stl" scale="3 3 3"/>
+        <mesh filename="${mesh_uri}/Blade_4.stl" scale="${s} ${s} ${s}"/>
       </geometry>
       <material name="blade4"><color rgba="0.9 0.4 0.1 1"/></material>
@@ -404,9 +404,9 @@
     <parent link="rotor_link"/>
     <child link="tool_link"/>
-    <origin xyz="0 0 0.030" rpy="0 0 0"/>
+    <origin xyz="0 0 ${0.010*s}" rpy="0 0 0"/>
   </joint>
   <link name="tool_link">
     <visual>
-      <geometry><sphere radius="0.015"/></geometry>
+      <geometry><sphere radius="${0.005*s}"/></geometry>
       <material name="red"><color rgba="1 0 0 1"/></material>
     </visual>
