Commit message: Corrige le bloc de collision detache + axes de rotation de la tete
Le 'bloc bleu' flottant dans RViz/Gazebo etait le cluster des geometries de
collision (boites handles/tete, cylindre rotor) definies a l'origine des
links, alors que les meshes STL portent des coordonnees d'assemblage
(~0.63, 0.88, 1.28). Apres recentrage par hull_to_base, ce cluster se
retrouvait a ~1.4 m du robot.

- Collisions repositionnees sur les pieces reelles (origins en coords STL).
- joint1_head passe par l'axe reel de la tete (0.626, 0.857) : la tete
  tourne desormais sur elle-meme au lieu d'orbiter autour de l'origine STL.
- Visuels de head/rotor/blades compenses par l'offset inverse.
- Cylindre de collision du rotor elargi a l'impeller entier (r=0.045).

Co-Authored-By: Claude Fable 5 <noreply@anthropic.com>

File: mon_robot_description/urdf/mon_robot.urdf.xacro (robot description, xacro)
@@ -15,10 +15,11 @@
        trajectoire n'est commandee (seuls joint1_head/joint2_rotor bougent).
        Le lien "world" sert aussi de repere fixe en RViz.
-       world_to_hull origin z : hauteur du repere technique par rapport a l'eau (z=0). -->
+       world_to_hull origin z : hauteur du repere technique par rapport a l'eau (z=0).
+       z=0.13 place le bas du STL au contact visuel de la surface. -->
   <link name="world"/>
   <joint name="world_to_hull" type="fixed">
     <parent link="world"/>
     <child link="hull_link"/>
-    <origin xyz="0 0 0.15" rpy="0 0 0"/>
+    <origin xyz="0 0 0.13" rpy="0 0 0"/>
   </joint>
   <!-- ========== REPERE TECHNIQUE INVISIBLE ==========
@@ -77,4 +78,6 @@
     </visual>
     <collision>
+      <!-- Origine = position reelle du handle dans les coords d'assemblage STL -->
+      <origin xyz="${0.666*s} ${0.908*s} ${1.272*s}" rpy="0 0 0"/>
       <geometry><box size="${0.010*s} ${0.008*s} ${0.025*s}"/></geometry>
     </collision>
@@ -102,4 +105,6 @@
     </visual>
     <collision>
+      <!-- Origine = position reelle du handle dans les coords d'assemblage STL -->
+      <origin xyz="${0.586*s} ${0.908*s} ${1.272*s}" rpy="0 0 0"/>
       <geometry><box size="${0.010*s} ${0.008*s} ${0.025*s}"/></geometry>
     </collision>
@@ -269,9 +274,13 @@
     </inertial>
   </link>
-  <!-- ========== JOINT 1 — TETE (part2) ROTATION PRINCIPALE ========== -->
+  <!-- ========== JOINT 1 — TETE (part2) ROTATION PRINCIPALE ==========
+       L'axe passe par la position reelle de la tete dans les coords
+       d'assemblage STL (x=0.626, y=0.857) : la tete tourne sur elle-meme
+       au lieu d'orbiter autour de l'origine du STL. Les visuels du sous-
+       arbre compensent avec l'offset inverse. -->
   <joint name="joint1_head" type="revolute">
     <parent link="base_link"/>
     <child link="head_link"/>
-    <origin xyz="0 0 0" rpy="0 0 0"/>
+    <origin xyz="${0.626*s} ${0.857*s} ${1.351*s}" rpy="0 0 0"/>
     <axis xyz="0 0 1"/>
     <limit lower="-3.14159" upper="3.14159"
@@ -281,4 +290,5 @@
   <link name="head_link">
     <visual>
+      <origin xyz="${-0.626*s} ${-0.857*s} ${-1.351*s}" rpy="0 0 0"/>
       <geometry>
         <mesh filename="${mesh_uri}/part2.stl"
@@ -290,5 +300,5 @@
     </visual>
     <collision>
-      <origin xyz="0 0 0" rpy="0 0 0"/>
+      <origin xyz="0 0 ${0.010*s}" rpy="0 0 0"/>
       <geometry>
         <box size="${0.101*s} ${0.043*s} ${0.039*s}"/>
@@ -313,4 +323,5 @@
   <link name="rotor_link">
     <visual>
+      <origin xyz="${-0.626*s} ${-0.857*s} ${-1.351*s}" rpy="0 0 0"/>
       <geometry>
         <mesh filename="${mesh_uri}/Blade_1.stl"
@@ -322,5 +333,6 @@
     </visual>
     <collision>
-      <geometry><cylinder radius="${0.015*s}" length="${0.006*s}"/></geometry>
+      <!-- Cylindre englobant l'impeller entier (les 4 pales, rayon ~0.045) -->
+      <geometry><cylinder radius="${0.045*s}" length="${0.006*s}"/></geometry>
     </collision>
     <inertial>
@@ -338,4 +350,5 @@
   <link name="blade2_link">
     <visual>
+      <origin xyz="${-0.626*s} ${-0.857*s} ${-1.351*s}" rpy="0 0 0"/>
       <geometry>
         <mesh filename="${mesh_uri}/Blade_2.stl" scale="${s} ${s} ${s}"/>
@@ -356,4 +369,5 @@
   <link name="blade3_link">
     <visual>
+      <origin xyz="${-0.626*s} ${-0.857*s} ${-1.351*s}" rpy="0 0 0"/>
       <geometry>
         <mesh filename="${mesh_uri}/Blade_3.stl" scale="${s} ${s} ${s}"/>
@@ -374,4 +388,5 @@
   <link name="blade4_link">
     <visual>
+      <origin xyz="${-0.626*s} ${-0.857*s} ${-1.351*s}" rpy="0 0 0"/>
       <geometry>
         <mesh filename="${mesh_uri}/Blade_4.stl" scale="${s} ${s} ${s}"/>
